File: IV6Thingie.kicad_sch (KiCad schematic)
At the start: 29 parts, among them J1 5V IN, SW1 Hour, SW2 Minute, SW3 Set, SW4 12/24, U1 ИВ-6, U10 ИВ-6, U13 DS1302+, U14 ИВ-6, U17 ИВ-6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

Commit message: clean up schema
Other:
- company: (none) -> Dave Hamilton
- title: (none) -> IV6 Thingie
- moved on the sheet: BT1, C12, D1, J1, R2, RN1, RN2, RN7, SW1, SW2, SW3, SW4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
